File: receiverV3/receiverV3.kicad_sch (KiCad schematic)
At the start: 25 parts, among them J1 Raspberry_Pi_4, J2 SM04B-SRSS-TB, J3 S2B-PH-SM4-TB, U1 Teensy4.0, U2 AP63300WU-7_mod

Commit message: add teensy4.1 version of receiver
Connections:
- net BUSY: now also U1.21 (14_A0_TX3_SPDIF_OUT); no longer U1.24 (17_A3_TX4_SDA1)
- net DIO1: now also U1.23 (16_A2_RX4_SCL1); no longer U1.22 (15_A1_RX3_SPDIF_IN)
- net GPS_STBY: now also U1.24 (17_A3_TX4_SDA1); no longer U1.21 (14_A0_TX3_SPDIF_OUT)
- net LO_RST: now also U1.9 (7_RX2_OUT1A); no longer U1.7 (5_IN2)
- net MOD_6_MULT: now also U1.6 (4_BCLK2); no longer U1.9 (7_RX2_OUT1A)
- net MOD_8_MULT: now also U1.7 (5_IN2); no longer U1.10 (8_TX2_IN1)
- net RAD_PWR: now also U1.22 (15_A1_RX3_SPDIF_IN); no longer U1.23 (16_A2_RX4_SCL1)
- no-connect marks 13 -> 15
Changed lines of the file:
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@@
+	)
+	(no_connect
+		(at 90.17 69.85)
 	)
 	(no_connect
@@
 		(at 179.07 101.6)
 	)
+	(no_connect
+		(at 80.01 69.85)
+	)
 	(wire
 		(pts
@@
 	(wire
 		(pts
-			(xy 77.47 69.85) (xy 90.17 69.85)
-		)
-		(stroke
-			(width 0)
-			(type default)
-		)
-	)
-	(wire
-		(pts
 			(xy 83.82 80.01) (xy 90.17 80.01)
 		)
@@
 	(wire
 		(pts
+			(xy 77.47 67.31) (xy 90.17 67.31)
+		)
+		(stroke
+			(width 0)
+			(type default)
+		)
+	)
+	(wire
+		(pts
 			(xy 223.52 78.74) (xy 238.76 78.74)
 		)
@@
 	(wire
 		(pts
+			(xy 77.47 59.69) (xy 90.17 59.69)
+		)
+		(stroke
+			(width 0)
+			(type default)
+		)
+	)
+	(wire
+		(pts
 			(xy 83.82 49.53) (xy 90.17 49.53)
 		)
@@
 	(wire
 		(pts
+			(xy 82.55 100.33) (xy 90.17 100.33)
+		)
+		(stroke
+			(width 0)
+			(type default)
+		)
+	)
+	(wire
+		(pts
+			(xy 83.82 113.03) (xy 90.17 113.03)
+		)
+		(stroke
+			(width 0)
+			(type default)
+		)
+	)
+	(wire
+		(pts
 			(xy 77.47 62.23) (xy 90.17 62.23)
 		)
@@
 	(wire
 		(pts
-			(xy 82.55 100.33) (xy 90.17 100.33)
-		)
-		(stroke
-			(width 0)
-			(type default)
-		)
-	)
-	(wire
-		(pts
-			(xy 83.82 113.03) (xy 90.17 113.03)
-		)
-		(stroke
-			(width 0)
-			(type default)
-		)
-	)
-	(wire
-		(pts
 			(xy 39.37 148.59) (xy 55.88 148.59)
 		)
@@
 	(wire
 		(pts
+			(xy 168.91 71.12) (xy 179.07 71.12)
+		)
+		(stroke
+			(width 0)
+			(type default)
+		)
+	)
+	(wire
+		(pts
+			(xy 223.52 104.14) (xy 240.03 104.14)
+		)
+		(stroke
+			(width 0)
+			(type default)
+		)
+	)
+	(wire
+		(pts
+			(xy 223.52 66.04) (xy 231.14 66.04)
+		)
+		(stroke
+			(width 0)
+			(type default)
+		)
+	)
+	(wire
+		(pts
 			(xy 77.47 64.77) (xy 90.17 64.77)
-		)
-		(stroke
-			(width 0)
-			(type default)
-		)
-	)
-	(wire
-		(pts
-			(xy 168.91 71.12) (xy 179.07 71.12)
-		)
-		(stroke
-			(width 0)
-			(type default)
-		)
-	)
-	(wire
-		(pts
-			(xy 223.52 104.14) (xy 240.03 104.14)
-		)
-		(stroke
-			(width 0)
-			(type default)
-		)
-	)
-	(wire
-		(pts
-			(xy 223.52 66.04) (xy 231.14 66.04)
-		)
-		(stroke
-			(width 0)
-			(type default)
-		)
-	)
-	(wire
-		(pts
-			(xy 77.47 67.31) (xy 90.17 67.31)
 		)
 		(stroke
@@
 		)
 	)
+	(label "MOD_6_MULT"
+		(at 77.47 59.69 0)
+		(effects
+			(font
+				(size 1.27 1.27)
+			)
+			(justify left bottom)
+		)
+	)
 	(label "CS0"
 		(at 83.82 74.93 0)
@@
 		)
 	)
-	(label "MOD_8_MULT"
-		(at 77.47 69.85 0)
-		(effects
-			(font
-				(size 1.27 1.27)
-			)
-			(justify left bottom)
-		)
-	)
 	(label "MOSI"
 		(at 168.91 86.36 0)
@@
 		)
 	)
+	(label "RAD_PWR"
+		(at 82.55 100.33 0)
+		(effects
+			(font
+				(size 1.27 1.27)
+			)
+			(justify left bottom)
+		)
+	)
+	(label "LO_RST"
+		(at 77.47 67.31 0)
+		(effects
+			(font
+				(size 1.27 1.27)
+			)
+			(justify left bottom)
+		)
+	)
 	(label "MOD_RST"
 		(at 227.33 81.28 0)
@@
 		)
 	)
-	(label "MOD_6_MULT"
-		(at 77.47 67.31 0)
-		(effects
-			(font
-				(size 1.27 1.27)
-			)
-			(justify left bottom)
-		)
-	)
 	(label "RX_ALT"
 		(at 83.82 49.53 0)
@@
 		)
 	)
-	(label "DIO1"
-		(at 82.55 100.33 0)
-		(effects
-			(font
-				(size 1.27 1.27)
-			)
-			(justify left bottom)
-		)
-	)
 	(label "SCK"
 		(at 168.91 91.44 0)
@@
 		)
 	)
-	(label "GPS_STBY"
-		(at 82.55 97.79 0)
-		(effects
-			(font
-				(size 1.27 1.27)
-			)
-			(justify left bottom)
-		)
-	)
-	(label "LO_RST"
-		(at 77.47 62.23 0)
-		(effects
-			(font
-				(size 1.27 1.27)
-			)
-			(justify left bottom)
-		)
-	)
 	(label "MISO"
 		(at 83.82 80.01 0)
@@
 		)
 	)
+	(label "MOD_8_MULT"
+		(at 77.47 62.23 0)
+		(effects
+			(font
+				(size 1.27 1.27)
+			)
+			(justify left bottom)
+		)
+	)
+	(label "SCL"
+		(at 83.82 110.49 0)
+		(effects
+			(font
+				(size 1.27 1.27)
+			)
+			(justify left bottom)
+		)
+	)
+	(label "CS0"
+		(at 227.33 91.44 0)
+		(effects
+			(font
+				(size 1.27 1.27)
+			)
+			(justify left bottom)
+		)
+	)
+	(label "RX"
+		(at 83.82 115.57 0)
+		(effects
+			(font
+				(size 1.27 1.27)
+			)
+			(justify left bottom)
+		)
+	)
+	(label "Enable"
+		(at 86.36 162.56 0)
+		(effects
+			(font
+				(size 1.27 1.27)
+			)
+			(justify left bottom)
+		)
+	)
+	(label "MOD_6_MULT"
+		(at 227.33 109.22 0)
+		(effects
+			(font
+				(size 1.27 1.27)
+			)
+			(justify left bottom)
+		)
+	)
+	(label "TX"
+		(at 83.82 113.03 0)
+		(effects
+			(font
+				(size 1.27 1.27)
+			)
+			(justify left bottom)
+		)
+	)
+	(label "RX"
+		(at 227.33 71.12 0)
+		(effects
+			(font
+				(size 1.27 1.27)
+			)
+			(justify left bottom)
+		)
+	)
+	(label "CS1"
+		(at 227.33 93.98 0)
+		(effects
+			(font
+				(size 1.27 1.27)
+			)
+			(justify left bottom)
+		)
+	)
 	(label "MOD_RST"
 		(at 77.47 64.77 0)
@@
 		)
 	)
-	(label "SCL"
-		(at 83.82 110.49 0)
-		(effects
-			(font
-				(size 1.27 1.27)
-			)
-			(justify left bottom)
-		)
-	)
-	(label "CS0"
-		(at 227.33 91.44 0)
-		(effects
-			(font
-				(size 1.27 1.27)
-			)
-			(justify left bottom)
-		)
-	)
-	(label "RX"
-		(at 83.82 115.57 0)
-		(effects
-			(font
-				(size 1.27 1.27)
-			)
-			(justify left bottom)
-		)
-	)
-	(label "Enable"
-		(at 86.36 162.56 0)
-		(effects
-			(font
-				(size 1.27 1.27)
-			)
-			(justify left bottom)
-		)
-	)
-	(label "MOD_6_MULT"
-		(at 227.33 109.22 0)
-		(effects
-			(font
-				(size 1.27 1.27)
-			)
-			(justify left bottom)
-		)
-	)
-	(label "TX"
-		(at 83.82 113.03 0)
-		(effects
-			(font
-				(size 1.27 1.27)
-			)
-			(justify left bottom)
-		)
-	)
-	(label "RAD_PWR"
+	(label "GPS_STBY"
+		(at 83.82 105.41 0)
+		(effects
+			(font
+				(size 1.27 1.27)
+			)
+			(justify left bottom)
+		)
+	)
+	(label "DIO1"
 		(at 83.82 102.87 0)
-		(effects
-			(font
-				(size 1.27 1.27)
-			)
-			(justify left bottom)
-		)
-	)
-	(label "RX"
-		(at 227.33 71.12 0)
-		(effects
-			(font
-				(size 1.27 1.27)
-			)
-			(justify left bottom)
-		)
-	)
-	(label "CS1"
-		(at 227.33 93.98 0)
 		(effects
 			(font
@@
 	)
 	(label "BUSY"
-		(at 83.82 105.41 0)
-		(effects
-			(font
+		(at 82.55 97.79 0)
+		(effects
+			(font
