File: receiverV5/receiverV5.kicad_sch (KiCad schematic)
At the start: 31 parts, among them J1 Raspberry_Pi_4, J3 S2B-PH-SM4-TB, J4 S2B-PH-SM4-TB, U2 AP63300WU-7_mod, U3 Teensy4.1

Commit message: update receiver repo
Parts:
- removed C3: 100n, Capacitor_SMD:C_0402_1005Metric, symbol Device:C_Small
- removed C4, C5: 22u, Capacitor_SMD:C_0402_1005Metric_Pad0.74x0.62mm_HandSolder, symbol Device:C_Small
- removed C6: 47p, Capacitor_SMD:C_0402_1005Metric_Pad0.74x0.62mm_HandSolder, symbol Device:C_Small
- removed C7, C9: 100n, Capacitor_SMD:C_0402_1005Metric_Pad0.74x0.62mm_HandSolder, symbol Device:C_Small
- removed L1: 6.8uH, Bourns_induct:IND_SRP5050FA-5R6M_BRN_mod, symbol Device:L_Small
- removed R1, R2: 100k, Resistor_SMD:R_0402_1005Metric_Pad0.72x0.64mm_HandSolder, symbol Device:R_Small_US
- removed R3: 162k, Resistor_SMD:R_0402_1005Metric_Pad0.72x0.64mm_HandSolder, symbol Device:R_US
- removed R4: 31.1k, Resistor_SMD:R_0402_1005Metric, symbol Device:R_US
- removed U2: AP63300WU-7_mod, footprints:SOIC_05WU-7_DIO-L_mod, symbol AP63300WU-7:AP63300WU-7_mod
- added J2: adafruitpwr1000, adafruit:adafruit powerboost 1000, symbol adafruit_power1000:adafruitpwr1000
- C1: footprint Capacitor_SMD:C_0603_1608Metric -> Capacitor_SMD:C_1206_3216Metric_Pad1.33x1.80mm_HandSolder; Description_1 Capacitor -> (none); MANUFACTURER Murata Electronics -> (none); Manufacturer_part_number GRT319R6YA106KE01D -> (none)
- C10, C8: value 1u -> 10u; footprint Capacitor_SMD:C_0603_1608Metric_Pad1.08x0.95mm_HandSolder -> Capacitor_SMD:C_1206_3216Metric_Pad1.33x1.80mm_HandSolder
- C2: value 100n -> 10u; footprint Capacitor_SMD:C_0402_1005Metric -> Capacitor_SMD:C_1206_3216Metric_Pad1.33x1.80mm_HandSolder; Description_1 Capacitor -> (none); MANUFACTURER Taiyo Yuden -> (none); Manufacturer_part_number GMK107BJ104KAHT -> (none)
- H1, H2, H3, H4: footprint TF:MountingHole_3mm_rec -> receiverBoard:mountinghole3mm
- H5: symbol Mechanical:MountingHole -> receiverBoard:mountinghole4mm
- H6, H7, H8: footprint TF:MountingHole_4mm_t4 -> receiverBoard:mountinghole4mm
- J1: footprint TF:PinHeader_2x20_P2.54mm_Vertical_receiver -> Connector_PinHeader_2.54mm:PinHeader_2x20_P2.54mm_Vertical
- J3, J4: footprint JST PH 2pin:CONN_S2B-PH-SM4-TB_JST -> JST2pin:CONN_S2B-PH-SM4-TB_JST_mod2
- J5: renamed from On/Off/switch1; footprint JST PH 2pin:CONN_S2B-PH-SM4-TB_JST_no_circle -> JST2pin:CONN_S2B-PH-SM4-TB_JST_mod2
- R5, R6: value 4.7k -> 3.3k; footprint Resistor_SMD:R_0402_1005Metric -> Resistor_SMD:R_1206_3216Metric_Pad1.30x1.75mm_HandSolder
Connections:
- net Enable is gone; now on net GND: J5.1
- net +5V: now also C1.2, C2.1, J2.8 (5V)
- net GND: now also C1.1, J3.1, J2.5 (GND), J2.7 (GND); no longer C1.2, J3.2
- net VBUS: now also J3.2, J2.1 (USB_PWR); no longer C1.1, C2.1, J3.1
- net GPS_RST: now reaches J1.22 (D25)
- net GPS_RST: now also U3.18 (26_A12_MOSI1)
- net STANDBY_GPS: now reaches J1.32 (DP12)
- net STANDBY_GPS: now also U3.8 (6_OUT1D)
- net GPS_RST_MAX_7Q: now reaches J1.33 (GP13)
- net GPS_RST_MAX_7Q: now also U3.7 (5_IN2)
- net STANDBY_GPS_MAX_7Q: now reaches J1.35 (GP19/SPI1_MISO)
- net STANDBY_GPS_MAX_7Q: now also U3.6 (4_BCLK2)
- net PWR_EN: now reaches J5.2
- net PWR_EN: now also J2.4 (EN)
- net BUSY: no longer names the net of J1.7 (DP4)
- net BUSY: no longer U3.22 (30_CRX3)
- net CS0 renamed SPI_CS0
- net CS1 renamed GPIO7_SX1302
- net DIO1: no longer names the net of U3.25 (33_MCLK2)
- net DIO1: no longer J1.11 (DP17)
- net GPS_STBY: no longer names the net of J1.13 (DP27)
- net GPS_STBY: no longer U3.23 (31_CTX3)
- net LO_RST: no longer names the net of J1.15 (DP22)
- net LO_RST: no longer U3.19 (27_A13_SCK1)
- net MOD_6_MULT: no longer names the net of J1.38 (DP20/SPI1_MOSI)
- net MOD_6_MULT: no longer U3.4 (2_OUT2)
- net MOD_8_MULT: no longer names the net of J1.36 (DP16/SPI1_CS0)
- net MOD_8_MULT: no longer U3.5 (3_LRCLK2)
- net MOD_RST: no longer names the net of J1.16 (D23)
- net MOD_RST: no longer U3.18 (26_A12_MOSI1)
- net RAD_PWR: no longer names the net of J1.12 (D18)
- net RAD_PWR: no longer U3.24 (32_OUT1B)
- net RX_ALT: no longer names the net of U3.2 (0_RX1_CRX2_CS1)
- net TX_ALT: no longer names the net of U3.3 (1_TX1_CTX2_MISO1)
- new net RESET_5146: J1.11 (DP17), U3.19 (27_A13_SCK1)
- no-connect marks 13 -> 16
Other:
- moved on the sheet: C10, C8, J1, J5
