File: receiver7RP2350V5/receiver7RP2350V5.kicad_pcb (KiCad board)
At the start: 4 copper layers, 48 x 78.3 mm, 70 parts, among them J10 S2B-PH-SM4-TB, J2 NT4R1600, J3 NT4R1600, J4 S2B-PH-SM4-TB, J6 MM60-52B1-E1-R650, J7 USB4105-GF-A, J8 S2B-PH-SM4-TB, U1 RP2354_60QFN, U2 USBLC6-2SC6, U4 MP2664GG-0000-Z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

Commit message: working drc for v5
Parts:
- moved J10 3.15 mm to (94.5, 128.9)
- moved D2 1.63 mm to (106.4, 122.1)
- moved J4 1.62 mm to (106.5, 128.9)
- moved H5 0.20 mm to (117.8, 85.6)
- turned C11 to 45 degrees
Routing:
- net Net-(J10-Pad2): track 6.55 -> 9.99 mm
- net /V_EN: track 26.6 -> 30.0 mm
- net +3V3: track 101.2 -> 98.2 mm
- net /VBUS: track 8.43 -> 10.1 mm
- net GND: track 58.3 -> 57.2 mm, vias 120 -> 143
- net /SX1261_BUSY: track 44.9 -> 43.9 mm
